File: ducktape.kicad_pcb (KiCad board)
At the start: 2 copper layers, 65 x 18 mm, 22 parts, among them J1 SSD1306, J2 USB_A, J3 USB_C_Receptacle_USB2.0_16P, J4 ARM, U2 W25Q16JVSSIQ, U3 RT9013-33GB, U4 ESP32-S3-MINI-1U

Commit message: finish pcb and generate gerbers
Parts:
- removed C5: 1uF, Capacitor_SMD:C_0402_1005Metric
- added C8: 1uF, Capacitor_SMD:C_0402_1005Metric, F.Cu at (136.5, 64.0)
- added G1: LOGO, asset_lib:nl_bw, F.Cu at (117.5, 52.0)
- added REF1: MountingHole_2.2mm_M2, MountingHole:MountingHole_2.2mm_M2, F.Cu at (110.0, 51.5)
- added REF1: MountingHole_2.2mm_M2, MountingHole:MountingHole_2.2mm_M2, F.Cu at (110.0, 66.5)
- J1: footprint Connector_PinSocket_2.54mm:PinSocket_1x04_P2.54mm_Vertical_SMD_Pin1Left -> Connector_PinSocket_2.54mm:PinSocket_1x04_P2.54mm_Vertical
- moved C4 146.5 mm to (156.0, 63.8), turned to 180 degrees
- moved R2 144.6 mm to (156.0, 62.0), turned to -90 degrees
- moved C3 143.6 mm to (156.0, 66.0), turned to 180 degrees
- moved J1 134.0 mm to (126.7, 52.0), turned to 90 degrees
- moved C6 133.4 mm to (125.0, 59.5), turned to -90 degrees
- moved R3 130.8 mm to (105.5, 53.0), turned to 180 degrees
- moved R1 129.3 mm to (135.0, 64.0), turned to -90 degrees
- moved C7 127.0 mm to (112.5, 61.5)
- moved R5 126.8 mm to (113.5, 64.0), turned to 180 degrees
- moved C2 125.5 mm to (115.5, 55.0), turned to -90 degrees
- moved C1 121.7 mm to (115.5, 57.5), turned to 90 degrees
- moved R4 120.8 mm to (104.0, 65.0), turned to 180 degrees
- moved S2 118.8 mm to (121.8, 63.5), turned to 90 degrees
- moved J4 112.9 mm to (128.0, 64.5), turned to 90 degrees
- moved S1 112.3 mm to (117.0, 63.5), turned to 90 degrees
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Connections:
- net /USP_DP renamed /USB_DP
- C1 pad 2: +3.3V -> +3V3
- C3 pad 2: +3.3V -> +3V3
- C4 pad 2: +3.3V -> +3V3
- C6 pad 1: +3.3V -> +3V3
- J1 pad 2: +3.3V -> +3V3
- R1 pad 1: +3.3V -> +3V3
- R2 pad 1: +3.3V -> +3V3
- R2 pad 2: GND -> Net-(U4-IO0)
- S1 pad 4: GND -> Net-(U4-IO0)
- U2 pad 3: +3.3V -> +3V3
- U2 pad 7: +3.3V -> +3V3
- U2 pad 8: +3.3V -> +3V3
- U3 pad 5: +3.3V -> +3V3
- U4 pad 3: +3.3V -> +3V3
- U4 pad 4: GND -> Net-(U4-IO0)
Routing:
- net /USB_DP: track 0.00 -> 105.5 mm, vias 0 -> 2
- net /USB_DM: track 0.00 -> 83.3 mm, vias 0 -> 3
- net +3V3: track 0.00 -> 72.9 mm, vias 0 -> 2
- net +5V: track 0.00 -> 65.8 mm, vias 0 -> 2
- net Net-(U4-IO0): track 0.00 -> 41.2 mm, vias 0 -> 2
- net /RGB_LED: track 0.00 -> 36.1 mm, vias 0 -> 2
- net /FLASH_CLK: track 0.00 -> 33.5 mm, vias 0 -> 2
- net /FLASH_MISO: track 0.00 -> 32.6 mm, vias 0 -> 2
- net /FLASH_CS: track 0.00 -> 31.3 mm, vias 0 -> 2
- net Net-(J4-Pin_1): track 0.00 -> 27.5 mm, vias 0 -> 1
- net /DISP_SCL: track 0.00 -> 22.8 mm, vias 0 -> 1
- net /FLASH_MOSI: track 0.00 -> 21.8 mm, vias 0 -> 2
- net /DISP_SDA: track 0.00 -> 19.7 mm, vias 0 -> 1
- net Net-(U4-EN): track 0.00 -> 17.2 mm
- net GND: track 0.00 -> 10.7 mm, vias 0 -> 20
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- added copper zone on B.Cu, net GND
- added copper zone on F.Cu, net GND
Other:
- board size 65 x 18 mm -> 65 x 22 mm
