File: ducktape.kicad_sch (KiCad schematic)
At the start: 22 parts, among them J1 SSD1306, J2 USB_A, J3 USB_C_Receptacle_USB2.0_16P, J4 ARM, U2 W25Q16JVSSIQ, U3 RT9013-33GB, U4 ESP32-S3-MINI-1U

Commit message: finish pcb and generate gerbers
Parts:
- removed C5: 1uF, Capacitor_SMD:C_0402_1005Metric, symbol Device:C_Small
- added C8: 1uF, Capacitor_SMD:C_0402_1005Metric, symbol Device:C_Small
- J1: footprint Connector_PinSocket_2.54mm:PinSocket_1x04_P2.54mm_Vertical_SMD_Pin1Left -> Connector_PinSocket_2.54mm:PinSocket_1x04_P2.54mm_Vertical
Connections:
- net +3.3V is gone; now on net +3V3: C1.2, C3.2, C4.2, C6.1, J1.2 (Pin_2), R1.1, R2.1, U2.3 (~{WP}(IO2)), U2.7 (~{HOLD}/RESET(IO3)), U2.8 (VCC), U3.5 (VOUT), U4.3 (3V3)
- net GND: now also C8.1; no longer R2.2, S1.4, U4.4 (IO0)
- net at R1.2, S2.4, U4.45 (EN): now also C8.2
- net USP_DP renamed USB_DP
- new net: R2.2, S1.4, U4.4 (IO0)
